File: PCB/IOBoardV0/Power.kicad_pcb (KiCad board)
At the start: 2 copper layers, 12 parts, among them J1 JACK_2P, J2 RJ45_2, J3 RJ45_2, J4 RJ45_2, J5 RJ45_2, J6 RJ45_2, J7 RJ45_2, J8 RJ45_2, J9 RJ45_2

Commit message: Add files via upload
Other:
- board outline added: 34.3 x 83.9 mm
Changed lines of the file:
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@@
     (links 70)
     (no_connects 0)
-    (area 22.530999 17.22501 56.209001 100.659001)
+    (area 22.047999 16.713999 56.438001 100.761001)
     (thickness 1.6)
-    (drawings 0)
+    (drawings 5)
     (tracks 122)
     (zones 0)
@@
     (visible_elements 7FFFFFFF)
     (pcbplotparams
-      (layerselection 3178497)
+      (layerselection 284196865)
       (usegerberextensions true)
-      (excludeedgelayer true)
+      (excludeedgelayer false)
       (linewidth 0.150000)
       (plotframeref false)
       (viasonmask false)
       (mode 1)
-      (useauxorigin false)
+      (useauxorigin true)
       (hpglpennumber 1)
       (hpglpenspeed 20)
@@
       (plotreference true)
       (plotvalue true)
-      (plotothertext true)
+      (plotothertext false)
       (plotinvisibletext false)
       (padsonsilk false)
@@
       (outputformat 1)
       (mirror false)
-      (drillshape 1)
+      (drillshape 0)
       (scaleselection 1)
-      (outputdirectory ""))
+      (outputdirectory /home/pi/Desktop/IOBoardV0/Gerber/Power/))
   )
   (net 0 "")
@@
     )
   )
+  (gr_line (start 22.098 16.764) (end 22.225 16.764) (angle 90) (layer Edge.Cuts) (width 0.1))
+  (gr_line (start 22.098 100.711) (end 22.098 16.764) (angle 90) (layer Edge.Cuts) (width 0.1))
+  (gr_line (start 56.388 100.711) (end 22.098 100.711) (angle 90) (layer Edge.Cuts) (width 0.1))
+  (gr_line (start 56.388 16.764) (end 56.388 100.711) (angle 90) (layer Edge.Cuts) (width 0.1))
+  (gr_line (start 22.225 16.764) (end 56.388 16.764) (angle 90) (layer Edge.Cuts) (width 0.1))
   (segment (start 46.482 46.863) (end 46.482 44.831) (width 0.254) (layer B.Cu) (net 1))
   (segment (start 46.482 44.831) (end 46.482 42.799) (width 0.254) (layer B.Cu) (net 1))
