File: PCB/IOBoardV0/Sensor_Level.kicad_pcb (KiCad board)
At the start: 2 copper layers, 28 parts, among them J1 RJ45_2, J2 RJ45_2, J3 RJ45_2, P1 CONN_8X2, U1 LM324, U2 LM324, U3 74LS148

Commit message: Add files via upload
Parts:
- moved R13 11.2 mm to (61.8, 37.0)
- moved R14 11.2 mm to (61.8, 40.3)
- moved R17 11.2 mm to (61.8, 30.4)
- moved C2 11.2 mm to (58.0, 24.3)
- moved D1 11.2 mm to (63.5, 19.7)
- moved J1 11.2 mm to (45.7, 21.0)
- moved J2 11.2 mm to (26.9, 21.0)
- moved P1 11.2 mm to (29.5, 37.2)
- moved R10 11.2 mm to (50.5, 57.8)
- moved R16 11.2 mm to (50.5, 40.4)
- moved R3 11.2 mm to (35.3, 79.8)
- moved R4 11.2 mm to (35.3, 83.1)
- moved R5 11.2 mm to (35.4, 61.0)
- moved R6 11.2 mm to (35.4, 57.5)
- moved R9 11.2 mm to (50.5, 61.1)
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Connections:
- J1 pad 3: (no net) -> VCC
- J1 pad 4: (no net) -> GND
- J1 pad 5: (no net) -> VCC
- J1 pad 6: (no net) -> GND
- J1 pad 7: (no net) -> VCC
- J1 pad 8: (no net) -> GND
Routing:
- net GND: track 175.6 -> 183.7 mm
- net VCC: track 225.3 -> 231.4 mm
- added copper zone on B.Cu, net (none)
- added copper zone on F.Cu, net (none)
- added copper zone on B.Cu, net GND
- added copper zone on F.Cu, net GND
- added copper zone on B.Cu, net VCC
Other:
- board outline added: 48.8 x 69.2 mm
