File: PCB/IOBoardV0/Sensor_Level.sch (KiCad schematic (older format))
At the start: 28 parts, among them J1 RJ45_2, J2 RJ45_2, J3 RJ45_2, P1 CONN_8X2, U1 LM324, U2 LM324, U3 74LS148

Commit message: Add files via upload
Connections:
- net GND: now also J1.4, J1.6, J1.8
- net VCC: now also J1.3, J1.5, J1.7
Changed lines of the file:
@@
 Sheet 1 1
 Title ""
-Date "23 apr 2020"
+Date "25 apr 2020"
 Rev ""
 Comp ""
@@
 	5050 8850 5050 6000
 Wire Wire Line
-	5350 900  5350 1100
+	5350 900  5350 1700
 Wire Wire Line
 	5350 1100 5900 1100
@@
 Wire Wire Line
 	5900 2700 5900 2800
+Wire Wire Line
+	5350 1300 5450 1300
+Connection ~ 5350 1100
+Wire Wire Line
+	5350 1500 5450 1500
+Connection ~ 5350 1300
+Wire Wire Line
+	5350 1700 5450 1700
+Connection ~ 5350 1500
+Wire Wire Line
+	5450 1400 5700 1400
+Connection ~ 5700 1400
+Wire Wire Line
+	5450 1600 5700 1600
+Connection ~ 5700 1600
+Wire Wire Line
+	5450 1800 5700 1800
+Connection ~ 5700 1800
 $EndSCHEMATC
