File: PCB/IOBoardV0/Actuator_Relay.kicad_pcb (KiCad board)
At the start: 2 copper layers, 15 parts, among them J1 RJ45_2, J2 RJ45_2, K1 RELAY_J9906, P1 KLEMENS_1, P2 CONN_8X2, Q1 BC557, Q2 2N2222A

Commit message: Add files via upload
Other:
- board outline added: 53.8 x 36.1 mm
Changed lines of the file:
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@@
     (area 16.180999 16.180999 70.179001 52.566711)
     (thickness 1.6)
-    (drawings 0)
+    (drawings 7)
     (tracks 152)
     (zones 0)
@@
   )
   (layers
-    (15 F.Cu signal hide)
+    (15 F.Cu signal)
     (0 B.Cu signal)
     (16 B.Adhes user)
@@
     (visible_elements 7FFFFFFF)
     (pcbplotparams
-      (layerselection 3178497)
+      (layerselection 284196865)
       (usegerberextensions true)
-      (excludeedgelayer true)
+      (excludeedgelayer false)
       (linewidth 0.150000)
       (plotframeref false)
       (viasonmask false)
       (mode 1)
-      (useauxorigin false)
+      (useauxorigin true)
       (hpglpennumber 1)
       (hpglpenspeed 20)
@@
       (plotreference true)
       (plotvalue true)
-      (plotothertext true)
+      (plotothertext false)
       (plotinvisibletext false)
       (padsonsilk false)
@@
       (outputformat 1)
       (mirror false)
-      (drillshape 1)
+      (drillshape 0)
       (scaleselection 1)
-      (outputdirectory ""))
+      (outputdirectory /home/pi/Desktop/IOBoardV0/Gerber/Actuator_Relay/))
   )
   (net 0 "")
@@
     )
   )
+  (gr_line (start 16.383 16.256) (end 16.383 16.383) (angle 90) (layer Edge.Cuts) (width 0.1))
+  (gr_line (start 70.231 16.256) (end 70.231 16.383) (angle 90) (layer Edge.Cuts) (width 0.1))
+  (gr_line (start 16.383 16.256) (end 70.231 16.256) (angle 90) (layer Edge.Cuts) (width 0.1))
+  (gr_line (start 16.383 16.51) (end 16.383 16.383) (angle 90) (layer Edge.Cuts) (width 0.1))
+  (gr_line (start 16.383 52.324) (end 16.383 16.51) (angle 90) (layer Edge.Cuts) (width 0.1))
+  (gr_line (start 70.231 52.324) (end 16.383 52.324) (angle 90) (layer Edge.Cuts) (width 0.1))
+  (gr_line (start 70.231 16.383) (end 70.231 52.324) (angle 90) (layer Edge.Cuts) (width 0.1))
   (segment (start 38.1 40.64) (end 39.878 40.64) (width 0.254) (layer F.Cu) (net 1))
   (segment (start 49.022 43.18) (end 50.8 43.18) (width 0.254) (layer F.Cu) (net 1))

Commit message: Add files via upload
Parts:
- added D2: DIODE, D3, F.Cu at (43.6, 47.5)
- moved D1 1.35 mm to (45.5, 41.0)
- moved P1 0.18 mm to (33.1, 21.5)
- moved K1 0.13 mm to (26.7, 40.8)
Routing:
- net N-0000022: track 37.4 -> 40.4 mm
- net VCC: track 70.9 -> 72.6 mm
- net N-000001: track 23.0 -> 21.4 mm
- net GND: track 42.0 -> 43.1 mm
- net N-000002: track 45.2 -> 44.3 mm
- net N-000005: track 40.2 -> 39.3 mm
- net N-000004: track 16.7 -> 17.4 mm
- added copper zone on B.Cu, net VCC
