File: PCB/IOBoardV0/IOBoardV0.kicad_pcb (KiCad board)
At the start: 2 copper layers, 28 parts, among them J2 RJ45_2, J3 RJ45_2, J4 RJ45_2, J5 RJ45_2, J6 RJ45_2, J7 RJ45_2, J8 RJ45_2, J9 RJ45_2, P1 RASPBERRY_HAT, U1 74LS04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

Commit message: Add files via upload
Other:
- board outline added: 87.8 x 79.9 mm
Changed lines of the file:
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@@
     (links 135)
     (no_connects 0)
-    (area 18.1864 13.640999 106.426001 93.26245)
+    (area 18.1864 13.157999 107.111001 93.218001)
     (thickness 1.6)
-    (drawings 0)
+    (drawings 5)
     (tracks 867)
     (zones 0)
@@
       (layerselection 284196865)
       (usegerberextensions true)
-      (excludeedgelayer true)
+      (excludeedgelayer false)
       (linewidth 0.150000)
       (plotframeref false)
@@
       (plotreference true)
       (plotvalue true)
-      (plotothertext true)
+      (plotothertext false)
       (plotinvisibletext false)
       (padsonsilk false)
@@
       (drillshape 0)
       (scaleselection 1)
-      (outputdirectory /home/pi/Desktop/IOBoardV0/Gerber/))
+      (outputdirectory /home/pi/Desktop/IOBoardV0/Gerber/IOBoardV0/))
   )
   (net 0 "")
@@
     )
   )
+  (gr_line (start 19.304 13.208) (end 19.558 13.208) (angle 90) (layer Edge.Cuts) (width 0.1))
+  (gr_line (start 19.304 93.091) (end 19.304 13.208) (angle 90) (layer Edge.Cuts) (width 0.1))
+  (gr_line (start 107.061 93.091) (end 19.304 93.091) (angle 90) (layer Edge.Cuts) (width 0.1))
+  (gr_line (start 107.061 13.208) (end 107.061 93.091) (angle 90) (layer Edge.Cuts) (width 0.1))
+  (gr_line (start 19.431 13.208) (end 107.061 13.208) (angle 90) (layer Edge.Cuts) (width 0.1))
   (via (at 55.88 63.881) (size 0.889) (layers F.Cu B.Cu) (net 0))
   (segment (start 58.42 45.72) (end 58.42 44.069) (width 0.254) (layer B.Cu) (net 1))

Commit message: Add files via upload
Connections:
- U6 pad 15: (no net) -> GND
Routing:
- net GND: track 307.5 -> 310.5 mm
Changed lines of the file:
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@@
 (kicad_pcb (version 3) (host pcbnew "(22-Jun-2014 BZR 4027)-stable")
   (general
-    (links 135)
+    (links 136)
     (no_connects 0)
     (area 18.1864 13.157999 107.111001 93.218001)
     (thickness 1.6)
     (drawings 5)
-    (tracks 867)
+    (tracks 869)
     (zones 0)
     (modules 28)
@@
   (net 16 /S7)
   (net 17 GND)
-  (net 18 N-0000012)
-  (net 19 N-0000013)
-  (net 20 N-0000014)
-  (net 21 N-0000015)
+  (net 18 N-0000011)
+  (net 19 N-0000012)
+  (net 20 N-0000013)
+  (net 21 N-0000014)
   (net 22 N-0000025)
   (net 23 N-0000029)
@@
   (net 41 N-0000079)
   (net 42 N-0000080)
-  (net 43 N-0000082)
-  (net 44 N-0000083)
-  (net 45 N-0000084)
-  (net 46 N-0000085)
-  (net 47 N-0000086)
-  (net 48 N-0000087)
+  (net 43 N-0000081)
+  (net 44 N-0000082)
+  (net 45 N-0000083)
+  (net 46 N-0000084)
+  (net 47 N-0000085)
+  (net 48 N-0000086)
   (net 49 N-000009)
   (net 50 VCC)
@@
     (add_net /S7)
     (add_net GND)
+    (add_net N-0000011)
     (add_net N-0000012)
     (add_net N-0000013)
     (add_net N-0000014)
-    (add_net N-0000015)
     (add_net N-0000025)
     (add_net N-0000029)
@@
     (add_net N-0000079)
     (add_net N-0000080)
+    (add_net N-0000081)
     (add_net N-0000082)
     (add_net N-0000083)
@@
     (add_net N-0000085)
     (add_net N-0000086)
-    (add_net N-0000087)
     (add_net N-000009)
     (add_net VCC)
@@
     (pad 2 thru_hole circle (at 3.81 0) (size 1.397 1.397) (drill 0.8128)
       (layers *.Cu *.Mask F.SilkS)
-      (net 46 N-0000085)
+      (net 46 N-0000084)
     )
     (model discret/resistor.wrl
@@
     (pad 1 thru_hole circle (at -3.81 0 180) (size 1.397 1.397) (drill 0.8128)
       (layers *.Cu *.Mask F.SilkS)
-      (net 18 N-0000012)
+      (net 18 N-0000011)
     )
     (pad 2 thru_hole circle (at 3.81 0 180) (size 1.397 1.397) (drill 0.8128)
@@
     (pad 2 thru_hole circle (at 3.81 0 180) (size 1.397 1.397) (drill 0.8128)
       (layers *.Cu *.Mask F.SilkS)
-      (net 18 N-0000012)
+      (net 18 N-0000011)
     )
     (model discret/resistor.wrl
@@
     (pad 2 thru_hole circle (at 3.81 0) (size 1.397 1.397) (drill 0.8128)
       (layers *.Cu *.Mask F.SilkS)
-      (net 47 N-0000086)
+      (net 47 N-0000085)
     )
     (model discret/resistor.wrl
@@
     (pad 1 thru_hole circle (at -3.81 0) (size 1.397 1.397) (drill 0.8128)
       (layers *.Cu *.Mask F.SilkS)
-      (net 45 N-0000084)
+      (net 45 N-0000083)
     )
     (pad 2 thru_hole circle (at 3.81 0) (size 1.397 1.397) (drill 0.8128)
@@
     (pad 18 thru_hole circle (at -3.81 -1.27 270) (size 1.524 1.524) (drill 1.016)
       (layers *.Cu *.Mask F.SilkS)
-      (net 18 N-0000012)
+      (net 18 N-0000011)
     )
     (pad 27 thru_hole circle (at 8.89 1.27 270) (size 1.524 1.524) (drill 1.016)
@@
     (pad 11 thru_hole oval (at 11.43 -3.81) (size 1.5748 2.286) (drill 0.8128)
       (layers *.Cu *.Mask F.SilkS)
-      (net 43 N-0000082)
+      (net 43 N-0000081)
     )
     (pad 12 thru_hole oval (at 8.89 -3.81) (size 1.5748 2.286) (drill 0.8128)
@@
     (pad 1 thru_hole rect (at -8.89 3.81) (size 1.5748 2.286) (drill 0.8128)
       (layers *.Cu *.Mask F.SilkS)
-      (net 20 N-0000014)
+      (net 20 N-0000013)
     )
     (pad 2 thru_hole oval (at -6.35 3.81) (size 1.5748 2.286) (drill 0.8128)
       (layers *.Cu *.Mask F.SilkS)
-      (net 21 N-0000015)
+      (net 21 N-0000014)
     )
     (pad 3 thru_hole oval (at -3.81 3.81) (size 1.5748 2.286) (drill 0.8128)
@@
     (pad 15 thru_hole oval (at -6.35 -3.81) (size 1.5748 2.286) (drill 0.8128)
       (layers *.Cu *.Mask F.SilkS)
+      (net 17 GND)
     )
     (pad 16 thru_hole oval (at -8.89 -3.81) (size 1.5748 2.286) (drill 0.8128)
@@
     (pad 12 thru_hole oval (at 1.27 -3.81) (size 1.5748 2.286) (drill 0.8128)
       (layers *.Cu *.Mask F.SilkS)
-      (net 21 N-0000015)
+      (net 21 N-0000014)
     )
     (pad 13 thru_hole oval (at -1.27 -3.81) (size 1.5748 2.286) (drill 0.8128)
       (layers *.Cu *.Mask F.SilkS)
-      (net 20 N-0000014)
+      (net 20 N-0000013)
     )
     (pad 14 thru_hole oval (at -3.81 -3.81) (size 1.5748 2.286) (drill 0.8128)
@@
     (pad 2 thru_hole oval (at -5.08 3.81) (size 1.5748 2.286) (drill 0.8128)
       (layers *.Cu *.Mask F.SilkS)
-      (net 44 N-0000083)
+      (net 44 N-0000082)
     )
     (pad 3 thru_hole oval (at -2.54 3.81) (size 1.5748 2.286) (drill 0.8128)
@@
     (pad 4 thru_hole oval (at 0 3.81) (size 1.5748 2.286) (drill 0.8128)
       (layers *.Cu *.Mask F.SilkS)
-      (net 48 N-0000087)
+      (net 48 N-0000086)
     )
     (pad 5 thru_hole oval (at 2.54 3.81) (size 1.5748 2.286) (drill 0.8128)
@@
     (pad 9 thru_hole oval (at 5.08 -3.81) (size 1.5748 2.286) (drill 0.8128)
       (layers *.Cu *.Mask F.SilkS)
-      (net 19 N-0000013)
+      (net 19 N-0000012)
     )
     (pad 10 thru_hole oval (at 2.54 -3.81) (size 1.5748 2.286) (drill 0.8128)
       (layers *.Cu *.Mask F.SilkS)
-      (net 48 N-0000087)
+      (net 48 N-0000086)
     )
     (pad 11 thru_hole oval (at 0 -3.81) (size 1.5748 2.286) (drill 0.8128)
@@
     (pad 12 thru_hole oval (at -2.54 -3.81) (size 1.5748 2.286) (drill 0.8128)
       (layers *.Cu *.Mask F.SilkS)
-      (net 44 N-0000083)
+      (net 44 N-0000082)
     )
     (pad 13 thru_hole oval (at -5.08 -3.81) (size 1.5748 2.286) (drill 0.8128)
@@
     (pad 1 thru_hole rect (at -7.62 3.81) (size 1.5748 2.286) (drill 0.8128)
       (layers *.Cu *.Mask F.SilkS)
-      (net 44 N-0000083)
+      (net 44 N-0000082)
     )
     (pad 2 thru_hole oval (at -5.08 3.81) (size 1.5748 2.286) (drill 0.8128)
@@
     (pad 1 thru_hole rect (at -7.62 3.81) (size 1.5748 2.286) (drill 0.8128)
       (layers *.Cu *.Mask F.SilkS)
-      (net 46 N-0000085)
+      (net 46 N-0000084)
     )
     (pad 2 thru_hole oval (at -5.08 3.81) (size 1.5748 2.286) (drill 0.8128)
@@
     (pad 4 thru_hole oval (at 0 3.81) (size 1.5748 2.286) (drill 0.8128)
       (layers *.Cu *.Mask F.SilkS)
-      (net 48 N-0000087)
+      (net 48 N-0000086)
     )
     (pad 5 thru_hole oval (at 2.54 3.81) (size 1.5748 2.286) (drill 0.8128)
@@
     (pad 8 thru_hole oval (at 7.62 -3.81) (size 1.5748 2.286) (drill 0.8128)
       (layers *.Cu *.Mask F.SilkS)
-      (net 44 N-0000083)
+      (net 44 N-0000082)
     )
     (pad 9 thru_hole oval (at 5.08 -3.81) (size 1.5748 2.286) (drill 0.8128)
@@
     (pad 10 thru_hole oval (at 2.54 -3.81) (size 1.5748 2.286) (drill 0.8128)
       (layers *.Cu *.Mask F.SilkS)
-      (net 43 N-0000082)
+      (net 43 N-0000081)
     )
     (pad 11 thru_hole oval (at 0 -3.81) (size 1.5748 2.286) (drill 0.8128)
@@
     (pad 1 thru_hole circle (at -3.81 0 180) (size 1.397 1.397) (drill 0.8128)
       (layers *.Cu *.Mask F.SilkS)
-      (net 46 N-0000085)
+      (net 46 N-0000084)
     )
     (model discret/diode.wrl
@@
     (pad 2 thru_hole circle (at 1.27 0 180) (size 1.6764 1.6764) (drill 0.8128)
       (layers *.Cu *.Mask F.SilkS)
-      (net 45 N-0000084)
+      (net 45 N-0000083)
     )
     (model discret/leds/led3_vertical_verde.wrl
@@
     (pad 1 thru_hole circle (at -1.27 0) (size 1.6764 1.6764) (drill 0.8128)
       (layers *.Cu *.Mask F.SilkS)
-      (net 47 N-0000086)
+      (net 47 N-0000085)
     )
     (pad 2 thru_hole circle (at 1.27 0) (size 1.6764 1.6764) (drill 0.8128)
       (layers *.Cu *.Mask F.SilkS)
-      (net 19 N-0000013)
+      (net 19 N-0000012)
     )
     (model discret/leds/led3_vertical_verde.wrl
@@
     (pad 1 thru_hole rect (at -1.27 0 180) (size 1.397 1.397) (drill 0.8128)
       (layers *.Cu *.Mask F.SilkS)
-      (net 46 N-0000085)
+      (net 46 N-0000084)
     )
     (pad 2 thru_hole circle (at 1.27 0 180) (size 1.397 1.397) (drill 0.8128)
@@
   (segment (start 72.771 81.915) (end 88.9 81.915) (width 0.254) (layer B.Cu) (net 16))
   (segment (start 72.517 82.169) (end 72.771 81.915) (width 0.254) (layer B.Cu) (net 16))
+  (segment (start 87.63 55.88) (end 87.63 58.674) (width 0.254) (layer F.Cu) (net 17))
+  (segment (start 87.63 58.674) (end 87.503 58.801) (width 0.254) (layer F.Cu) (net 17))
   (via (at 36.703 75.565) (size 0.889) (layers F.Cu B.Cu) (net 17))
   (segment (start 74.93 63.5) (end 79.883 63.5) (width 0.254) (layer F.Cu) (net 17))
